Commit message: test on robot works

File: security/iscoin_azz.urdf (robot description, URDF)
Before this commit: robot ur, 14 links, 13 joints
Links:
- link pen_link: geometry collision cylinder length=0.26 radius=0.032; visual cylinder length=0.26 radius=0.032
Joints:
- joint wrist_3-pen: origin xyz=0 0 0.1 rpy=0 0 0 -> xyz=0 0 0.125 rpy=0 0 0
